File: hardware/vextreme.kicad_pcb (KiCad board)
At the start: 2 copper layers, 48 x 66.1 mm, 49 parts, among them CON1 vectrex-edge-connector, J1 USB_C_Receptacle_USB2.0, J2 Conn_01x06_Male, U1 LM1117-3.3, U2 STM32F411RCTx, U3 74HC32, U4 SN74LVC8T245DB, U5 W25Q128, Y1 8MHz

Commit message: rename 'veccart' to 'stm32' for firmware and 'vextreme' for hardware, rename 'multicart' to 'menu'.
Parts:
- CON1: footprint veccart:vectrex-edge-connector-thinner-no-soldermask -> vextreme:vectrex-edge-connector-thinner-no-soldermask
- D10, D11, D12, D13, D4, D5, D6, D7, D8, D9: footprint veccart:LED-APA102-2020_6_REV_2 -> vextreme:LED-APA102-2020_6_REV_2
- J1: footprint veccart:USB_C_Receptacle_HRO_TYPE-C-31-M-12 -> vextreme:USB_C_Receptacle_HRO_TYPE-C-31-M-12
- hole1, hole3: footprint veccart:Mounting_Hole_D3.7mm -> vextreme:Mounting_Hole_D3.7mm
- hole2: footprint veccart:Mounting_Hole_D5.2mm -> vextreme:Mounting_Hole_D5.2mm
- hole4, hole5: footprint veccart:Mounting_Hole_D4.2mm -> vextreme:Mounting_Hole_D4.2mm
