File: hardware/vextreme.sch (KiCad schematic (older format))
At the start: 42 parts, among them CON1 vectrex-edge-connector, J1 USB_C_Receptacle_USB2.0, J2 Conn_01x06_Male, U1 LM1117-3.3, U2 STM32F411RCTx, U3 74HC32, U4 SN74LVC8T245DB, U5 W25Q128, Y1 8MHz

Commit message: rename 'veccart' to 'stm32' for firmware and 'vextreme' for hardware, rename 'multicart' to 'menu'.
Parts:
- CON1: footprint veccart:vectrex-edge-connector-thinner-no-soldermask -> vextreme:vectrex-edge-connector-thinner-no-soldermask; symbol veccart-rescue:vectrex-edge-connector-veccart-rescue -> vextreme-rescue:vectrex-edge-connector-vextreme-rescue
- D10, D11, D12, D13, D4, D5, D6, D7, D8, D9: footprint veccart:LED-APA102-2020_6_REV_2 -> vextreme:LED-APA102-2020_6_REV_2
- J1: footprint veccart:USB_C_Receptacle_HRO_TYPE-C-31-M-12 -> vextreme:USB_C_Receptacle_HRO_TYPE-C-31-M-12
Other:
- note added: "v0.3 Changelog\n——————————————————————\n- Fixed PCB fingers (removed soldermask ink around fingers, made them 8.8mm\n x 1.52mm, spaced 1.2mm from board edge, and 18.0mm from 3.6mm hole)\n- Increased hole sizes to 3.7mm, 4.2mm, 5.2mm\n- Made all pads on addressable LEDs the same size\n"
- note removed: "v0.2 Changelog\n——————————————————————\n- Replaced USB-B-mini with USB-C and centered USB on cart\n- Extended the PCB by 1.7 mm to get the USB-C connector as close to the case\n exterior as possible.\n- Widened the PCB to 48.0 mm so that there’s less side to side play in the cartridge slot.\n- Moved outer mounting holes into the proper locations\n- Reversed D3 and R4 order to get D3 closer to edg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"

Commit message: remove rescue library and merge all schematic parts into a common vextreme.lib
Parts:
- C1, C10, C11, C12, C13, C2, C3, C4, C5, C6, C7, C8, C9: symbol Device:C -> vextreme:C
- CON1: symbol vextreme-rescue:vectrex-edge-connector-vextreme-rescue -> vextreme:vectrex-edge-connector
- D1, D2: symbol Diode:MBR0520 -> vextreme:MBR0520
- D10, D11, D12, D13, D4, D5, D6, D7, D8, D9: symbol LED:APA102-2020 -> vextreme:APA102-2020
- D3: symbol Device:LED -> vextreme:LED
- J1: symbol Connector:USB_C_Receptacle_USB2.0 -> vextreme:USB_C_Receptacle_USB2.0
- J2: symbol Connector:Conn_01x06_Male -> vextreme:Conn_01x06_Male
- JP1: symbol Device:Jumper_NO_Small -> vextreme:Jumper_NO_Small
- R1, R2, R3, R4, R5, R6: symbol Device:R -> vextreme:R
- U1: symbol Regulator_Linear:LM1117-3.3 -> vextreme:LM1117-3.3
- U3: symbol 74xx:74LS32 -> vextreme:74LS32
- U4: symbol Gekkio_Logic_LevelTranslator:SN74LVC8T245DB -> vextreme:SN74LVC8T245DB
- U5: symbol X:W25Q128 -> vextreme:W25Q128
- Y1: symbol Device:Crystal -> vextreme:Crystal

Commit message: v0.3 Hardware Changes
    - moved vextreme symbol library into libs/ folder
    - renaming 'veccart' to 'vextreme' for hardware files
    - Generate v0.3 gerbers, pdf and BOM
    - Finish routing v0.3 PCB
    - Fixes #21, added VEXTREME logo to PCB
    - Also moved most components to the bottom side and unrouted to prepare for single-sided conversion
    - Fixes #18, Add ESD protection to USB
    - Fixes #36, add test points for power rails.  Also add VEC-5V to PA10 to detect when Vectrex is on/off
    - Fixes #15, replace U3 with a single OR gate and add optional R7 to omit U3 completely
    - add SW1 for programming, add SW2 for STM32 reset
    - adds 3-pin header for LED output
    - Fixes #13, move the debugging/serial port connector so it does not interfere with enclosure bosses
    - Fixes #9, R4 & D3 reference designators are swapped
    - Fixes #12, reduce from 10 to 4 LEDs
Parts:
- removed D10, D12, D4, D5, D6, D8: APA102-2020, vextreme:LED-APA102-2020_6_REV_2, symbol vextreme:APA102-2020
- removed U3: 74HC32, Package_SO:SOIC-14_3.9x8.7mm_P1.27mm, symbol vextreme:74LS32
- added J3: Conn_01x03_Male, Connector_PinHeader_2.54mm:PinHeader_1x03_P2.54mm_Vertical, symbol Connector:Conn_01x03_Male
- added JP2: Jumper_3_Bridged12, vextreme:SolderJumper-3_P1.3mm_Bridged12_RoundedPad1.0x1.5mm_NumberLabels, symbol Jumper:Jumper_3_Bridged12
- added R7: 0, Resistor_SMD:R_0805_2012Metric_Pad1.15x1.40mm_HandSolder, symbol Device:R
- added SP1: PA8, vextreme:SparePin_1x01_P2.54mm_Vertical, symbol Connector:TestPoint
- added SP2: PA13, vextreme:SparePin_1x01_P2.54mm_Vertical, symbol Connector:TestPoint
- added SP3: PA14, vextreme:SparePin_1x01_P2.54mm_Vertical, symbol Connector:TestPoint
- added SP4: PD2, vextreme:SparePin_1x01_P2.54mm_Vertical, symbol Connector:TestPoint
- added SW1: K3-1296S-E2, vextreme:SW_SPDT_K3-1296S-E2, symbol Switch:SW_SPST
- added SW2: TS-1002S-11526C, vextreme:SW_Push_1P1T_NO_6x6mm_H11.5mm, symbol Switch:SW_Push
- added TP1: V5V, TestPoint:TestPoint_Pad_D1.5mm, symbol Connector:TestPoint
- added TP2: 5V, TestPoint:TestPoint_Pad_D1.5mm, symbol Connector:TestPoint
- added TP3: GND, TestPoint:TestPoint_Pad_D1.5mm, symbol Connector:TestPoint
- added TP4: U5V, TestPoint:TestPoint_Pad_D1.5mm, symbol Connector:TestPoint
- added TP5: 3V3, TestPoint:TestPoint_Pad_D1.5mm, symbol Connector:TestPoint
- added U3: 74LVC1G32, vextreme:SOT-23-5_HandSoldering, symbol 74xGxx:74LVC1G32
- added U6: TPD4E02B04DQA, vextreme:USON-10_2.5x1.0mm_P0.5mm_passthrough, symbol vextreme:TPD4E02B04DQA_passthrough
- C13: value 47u -> 10u
- D4: renamed from D7; symbol vextreme:APA102-2020 -> LED:APA102-2020
- D5: renamed from D9; symbol vextreme:APA102-2020 -> LED:APA102-2020
- D6: renamed from D11; symbol vextreme:APA102-2020 -> LED:APA102-2020
- D7: renamed from D13; symbol vextreme:APA102-2020 -> LED:APA102-2020
- J2: value Conn_01x06_Male -> Conn_01x03_Male; footprint Connector_PinHeader_2.54mm:PinHeader_1x06_P2.54mm_Vertical -> Connector_PinHeader_2.54mm:PinHeader_1x03_P2.54mm_Vertical; symbol vextreme:Conn_01x06_Male -> Connector:Conn_01x03_Male
Connections:
- net labels added: NRST, PA8, USB-5V, VEC-5V
- net labels removed: C_VCC, SCLK_CONT, SDAT_CONT, USB-IN
- wire segments 138 -> 150
Other:
- note added: "/E"
- note added: "A15"
- note added: "JP2 normally connected (1-2) for SW2 to\nact as hard reset for STM32. If (1-2) cut\nand (2-3) soldered SW2 will be connected\nto pull PA8 low (should enable internal\npull-up) to use."
- note added: "v0.3 Changelog\n——————————————————————\n- Fixed PCB fingers (removed soldermask ink around fingers, made them 8.8mm\n x 1.52mm, spaced 1.2mm from board edge, and 18.0mm from 3.6mm hole)\n- Increased hole sizes to 3.7mm, 4.2mm, 5.2mm\n- Made all pads on addressable LEDs the same size\n- Remove D8 - D13, spacing remaining 4 LEDs evenly (13mm)\n- Change debugging header to 3-pin\n- Add 3-pin header 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"
- note removed: "v0.3 Changelog\n——————————————————————\n- Fixed PCB fingers (removed soldermask ink around fingers, made them 8.8mm\n x 1.52mm, spaced 1.2mm from board edge, and 18.0mm from 3.6mm hole)\n- Increased hole sizes to 3.7mm, 4.2mm, 5.2mm\n- Made all pads on addressable LEDs the same size\n"

Commit message: v0.4 Hardware Changes
- Increased length of SW2 to 12mm (TS-1002S-12026C)
- Changed SW1 to be the same as SW2
- Replaced J2 & J3 with a single 2x3 header that presses into place and holds
itself for soldering. Can use two separate 1x3 headers if desired.
- Replaced JP1 with a 1x2 header that presses into place for soldering.
- Added a micro 10-pin JTAG debugging header that doubles as USB Serial
adapter as well.
- Added a solderable jumper on V-NMI to be connected to one of PA8, which
also can be optionally connected to SW2.
- Added a diode for reverse polarity (cart upside down) on VEC_5V detect line. - Added a this side up label.
Parts:
- removed SW1: K3-1296S-E2, vextreme:SW_SPDT_K3-1296S-E2, symbol Switch:SW_SPST
- added D8: MBR0520, Diode_SMD:D_SOD-123, symbol Diode:MBR0520
- added J4: FTSH-105-01-F-DV-K, vextreme:CONN5X2_1.27, symbol Connector_Generic:Conn_02x05_Odd_Even
- added JP3: +3.3V Jumper, Jumper:SolderJumper-2_P1.3mm_Open_RoundedPad1.0x1.5mm, symbol Jumper:SolderJumper_2_Open
- added JP4: V-NMI Jumper, Jumper:SolderJumper-2_P1.3mm_Open_RoundedPad1.0x1.5mm, symbol Jumper:SolderJumper_2_Open
- added SW1: TS-1002S-12026C, vextreme:SW_Push_1P1T_NO_6x6mm_H12.0mm, symbol Switch:SW_Push
- J2, J3: footprint Connector_PinHeader_2.54mm:PinHeader_1x03_P2.54mm_Vertical -> vextreme:PinHeader_1x03_P2.54mm_Vertical_Odd_Even
- JP1: value Jumper_NO_Small -> Jumper; footprint Connector_PinHeader_2.54mm:PinHeader_1x02_P2.54mm_Vertical -> vextreme:PinHeader_1x02_P2.54mm_Vertical_Odd_Even
- SW2: value TS-1002S-11526C -> TS-1002S-12026C; footprint vextreme:SW_Push_1P1T_NO_6x6mm_H11.5mm -> vextreme:SW_Push_1P1T_NO_6x6mm_H12.0mm
Connections:
- net labels added: NMI, PA13, PA14, SWCLK, SWDIO
- wire segments 150 -> 175
- no-connect marks 0 -> 3
Other:
- note added: "CL = (C8 * C9)/(C8 + C9) + Cstray\n(324pF/36pF) + 4pF = 13pF\n(close to 12pF Y1 CL requirement)\n"
- note added: "v0.4 Changelog\n——————————————————————\n- Increased length of SW2 to 12mm (TS-1002S-12026C)\n- Changed SW1 to be the same as SW2\n- Replaced J2 & J3 with a single 2x3 header that presses into place and holds\n itself for soldering. Can use two separate 1x3 headers if desired.\n- Replaced JP1 with a 1x2 header that presses into place for soldering.\n- Added a micro 10-pin JTAG debugging header tha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"
- note removed: "CL = (C8 * C9)/(C8 + C9) + Cstray\n(324pF/36pF) + 4pF = 13pF (close to 12pF Y1 CL requirement)\n"
- moved on the sheet: D2, J2, JP2, SW2, TP1, TP2, TP5

Commit message: v0.5 Hardware Changes
- Added a location for a Wi-Fi module
- Changed J2 to support +5V for the Wi-Fi module
- Changed the artwork a bit and side up/down text
Parts:
- J2: value Conn_01x03_Male -> Conn_01x04_Male; footprint vextreme:PinHeader_1x03_P2.54mm_Vertical_Odd_Even -> vextreme:PinHeader_1x04_P2.54mm_Vertical_Odd_Even; symbol Connector:Conn_01x03_Male -> Connector:Conn_01x04_Male
- J4, JP1: Field4 (none) -> DNP
Connections:
- wire segments 175 -> 176
Other:
- note added: "v0.5 Changelog\n——————————————————————\n- Added a location for the Wi-Fi Module\n- Changed J2 to support +5V for the Wi-Fi Module\n- Changed the artwork a bit and side up/down text."
Changed lines of the file:
@@
 Sheet 1 1
 Title "VEXTREME Vectrex Multicart"
-Date "2020-09-11"
-Rev "v0.4"
+Date "2021-05-15"
+Rev "v0.5"
 Comp ""
 Comment1 ""
@@
 F 2 "vextreme:PinHeader_1x02_P2.54mm_Vertical_Odd_Even" H 2800 1450 50  0001 C CNN
 F 3 "~" H 2800 1450 50  0001 C CNN
+F 4 "DNP" V 2650 1300 50  0000 C CNN "Field4"
 	1    2800 1450
 	0    -1   -1   0
@@
 P_D7
 $Comp
-L Connector:Conn_01x03_Male J2
+L Connector:Conn_01x04_Male J2
 U 1 1 5D0ADA96
-P 10850 5100
-F 0 "J2" H 10900 5350 50  0000 R CNN
-F 1 "Conn_01x03_Male" H 11250 4900 50  0000 R CNN
-F 2 "vextreme:PinHeader_1x03_P2.54mm_Vertical_Odd_Even" H 10850 5100 50  0001 C CNN
-F 3 "~" H 10850 5100 50  0001 C CNN
-	1    10850 5100
+P 10850 5000
+F 0 "J2" H 10900 5250 50  0000 R CNN
+F 1 "Conn_01x04_Male" H 11250 4700 50  0000 R CNN
+F 2 "vextreme:PinHeader_1x04_P2.54mm_Vertical_Odd_Even" H 10850 5000 50  0001 C CNN
+F 3 "~" H 10850 5000 50  0001 C CNN
+	1    10850 5000
 	-1   0    0    -1
 $EndComp
@@
 	9750 5850 9850 5850
 Wire Wire Line
-	10350 5000 10650 5000
+	10350 4900 10650 4900
 $Comp
 L Connector:Conn_01x03_Male J3
@@
 Wire Wire Line
 	4650 5900 4600 5900
-$Comp
-L Graphic:Logo_Open_Hardware_Small #LOGO1
-U 1 1 5EE7732D
-P 7300 6850
-F 0 "#LOGO1" H 7300 7125 50  0001 C CNN
-F 1 "Logo_Open_Hardware_Small" H 7300 6625 50  0001 C CNN
-F 2 "" H 7300 6850 50  0001 C CNN
-F 3 "~" H 7300 6850 50  0001 C CNN
-	1    7300 6850
-	1    0    0    -1
-$EndComp
 Connection ~ 5800 3600
 Wire Wire Line
@@
 F 2 "vextreme:CONN5X2_1.27" H 8200 4650 50  0001 C CNN
 F 3 "~" H 8200 4650 50  0001 C CNN
+F 4 "DNP" H 8250 4350 50  0000 C CNN "Field4"
 	1    8200 4650
 	1    0    0    -1
@@
 Wire Wire Line
 	8000 5150 8500 5150
+Wire Wire Line
+	10350 5000 10650 5000
+$Comp
+L vextreme-rescue:+5V-vextreme-rescue #PWR0135
+U 1 1 60A19939
+P 10350 4900
+F 0 "#PWR0135" H 10350 4750 50  0001 C CNN
+F 1 "+5V" H 10350 5040 50  0000 C CNN
+F 2 "" H 10350 4900 50  0001 C CNN
+F 3 "" H 10350 4900 50  0001 C CNN
+	1    10350 4900
+	1    0    0    -1
+$EndComp
+$Comp
+L Graphic:Logo_Open_Hardware_Small #LOGO1
+U 1 1 5EE7732D
+P 7300 6850
+F 0 "#LOGO1" H 7300 7125 50  0001 C CNN
+F 1 "Logo_Open_Hardware_Small" H 7300 6625 50  0001 C CNN
+F 2 "Symbol:OSHW-Logo_5.7x6mm_SilkScreen" H 7300 6850 50  0001 C CNN
+F 3 "~" H 7300 6850 50  0001 C CNN
+	1    7300 6850
+	1    0    0    -1
+$EndComp
+Text Notes 7950 3500 0    50   ~ 0
+v0.5 Changelog\n——————————————————————\n- Added a location for the Wi-Fi Module\n- Changed J2 to support +5V for the Wi-Fi Module\n- Changed the artwork a bit and side up/down text.
 $EndSCHEMATC

Commit message: v1.0 Hardware Changes
- Bumped the version number
- I think that's all I did?? :D
Parts:
- CON1: symbol vextreme:vectrex-edge-connector -> vextreme-rescue:vectrex-edge-connector-vextreme-rescue-vextreme-rescue
Other:
- note added: "v0.5 Changelog (aka v1.0)\n——————————————————————\n- Added a location for the Wi-Fi Module\n- Changed J2 to support +5V for the Wi-Fi Module\n- Changed the artwork a bit and side up/down text."
- note removed: "v0.5 Changelog\n——————————————————————\n- Added a location for the Wi-Fi Module\n- Changed J2 to support +5V for the Wi-Fi Module\n- Changed the artwork a bit and side up/down text."
Changed lines of the file:
@@
 Sheet 1 1
 Title "VEXTREME Vectrex Multicart"
-Date "2021-05-15"
-Rev "v0.5"
+Date "2021-06-19"
+Rev "v1.0"
 Comp ""
 Comment1 ""
@@
 $EndDescr
 $Comp
-L vextreme:GND #PWR07
+L vextreme-rescue:GND-vextreme-rescue-vextreme-rescue #PWR07
 U 1 1 59F16914
 P 1700 5300
@@
 $EndComp
 $Comp
-L vextreme:GND #PWR0101
+L vextreme-rescue:GND-vextreme-rescue-vextreme-rescue #PWR0101
 U 1 1 5D00E463
 P 3850 6350
@@
 $EndComp
 $Comp
-L vextreme:GND #PWR0102
+L vextreme-rescue:GND-vextreme-rescue-vextreme-rescue #PWR0102
 U 1 1 5D00E892
 P 4600 6350
@@
 	4250 6200 4250 6350
 $Comp
-L vextreme:GND #PWR0103
+L vextreme-rescue:GND-vextreme-rescue-vextreme-rescue #PWR0103
 U 1 1 5D00F858
 P 4250 6350
@@
 USB-5V
 $Comp
-L vextreme:GND #PWR0105
+L vextreme-rescue:GND-vextreme-rescue-vextreme-rescue #PWR0105
 U 1 1 5D01B9D7
 P 5800 4750
@@
 $EndComp
 $Comp
-L vextreme:GND #PWR0106
+L vextreme-rescue:GND-vextreme-rescue-vextreme-rescue #PWR0106
 U 1 1 5D023148
 P 5550 5050
@@
 $EndComp
 $Comp
-L vextreme:+5V #PWR0112
+L vextreme-rescue:+5V-vextreme-rescue-vextreme-rescue #PWR0112
 U 1 1 5D05FE50
 P 7350 750
@@
 $EndComp
 $Comp
-L vextreme:+5V #PWR0117
+L vextreme-rescue:+5V-vextreme-rescue-vextreme-rescue #PWR0117
 U 1 1 5D06ED8C
 P 1350 1000
@@
 Connection ~ 4350 4750
 $Comp
-L vextreme:GND #PWR0119
+L vextreme-rescue:GND-vextreme-rescue-vextreme-rescue #PWR0119
 U 1 1 5D07FB9D
 P 4700 4850
@@
 	5550 5900 5550 6000
 $Comp
-L vextreme:GND #PWR0124
+L vextreme-rescue:GND-vextreme-rescue-vextreme-rescue #PWR0124
 U 1 1 5D0A1129
 P 5550 6000
@@
 $EndComp
 $Comp
-L vextreme:GND #PWR0126
+L vextreme-rescue:GND-vextreme-rescue-vextreme-rescue #PWR0126
 U 1 1 5D0F5289
 P 6050 3750
@@
 $EndComp
 $Comp
-L vextreme:+5V #PWR0127
+L vextreme-rescue:+5V-vextreme-rescue-vextreme-rescue #PWR0127
 U 1 1 5D0F55E9
 P 6050 3450
@@
 $EndComp
 $Comp
-L vextreme:+5V #PWR0128
+L vextreme-rescue:+5V-vextreme-rescue-vextreme-rescue #PWR0128
 U 1 1 5D0F60DC
 P 3850 5900
@@
 $EndComp
 $Comp
-L vextreme:GND #PWR0130
+L vextreme-rescue:GND-vextreme-rescue-vextreme-rescue #PWR0130
 U 1 1 5D0AE42B
 P 10350 5000
@@
 USB-5V
 $Comp
-L vextreme:GND #PWR0118
+L vextreme-rescue:GND-vextreme-rescue-vextreme-rescue #PWR0118
 U 1 1 5DEA6FB0
 P 1150 7400
@@
 $EndComp
 $Comp
-L vextreme:GND #PWR0131
+L vextreme-rescue:GND-vextreme-rescue-vextreme-rescue #PWR0131
 U 1 1 5DEA771E
 P 850 7400
@@
 	3250 6200 3100 6200
 $Comp
-L vextreme:GND #PWR0132
+L vextreme-rescue:GND-vextreme-rescue-vextreme-rescue #PWR0132
 U 1 1 5DF1039D
 P 3450 6100
@@
 	5100 3150 4950 3150
 $Comp
-L vextreme-rescue:GND-vextreme-rescue #PWR0139
+L vextreme-rescue:GND-vextreme-rescue-vextreme-rescue #PWR0139
 U 1 1 5E22D72D
 P 8100 6250
@@
 $EndComp
 $Comp
-L vextreme:+5V #PWR0140
+L vextreme-rescue:+5V-vextreme-rescue-vextreme-rescue #PWR0140
 U 1 1 5E22D733
 P 8100 5650
@@
 $EndComp
 $Comp
-L vextreme:vectrex-edge-connector CON1
+L vextreme-rescue:vectrex-edge-connector-vextreme-rescue-vextreme-rescue CON1
 U 1 1 59F1631A
 P 1800 3500
@@
 $EndComp
 $Comp
-L vextreme:GND #PWR0154
+L vextreme-rescue:GND-vextreme-rescue-vextreme-rescue #PWR0154
 U 1 1 5DEB047F
 P 7350 6300
@@
 $EndComp
 $Comp
-L vextreme:+5V #PWR0155
+L vextreme-rescue:+5V-vextreme-rescue-vextreme-rescue #PWR0155
 U 1 1 5DEB5A91
 P 7350 6000
@@
 $EndComp
 $Comp
-L vextreme-rescue:+5V-vextreme-rescue #PWR0152
+L vextreme-rescue:+5V-vextreme-rescue-vextreme-rescue #PWR0152
 U 1 1 5E24CDB0
 P 10150 5650
@@
 $EndComp
 $Comp
-L vextreme-rescue:GND-vextreme-rescue #PWR0151
+L vextreme-rescue:GND-vextreme-rescue-vextreme-rescue #PWR0151
 U 1 1 5E24CDAA
 P 10150 6250
@@
 $EndComp
 $Comp
-L vextreme-rescue:+5V-vextreme-rescue #PWR0148
+L vextreme-rescue:+5V-vextreme-rescue-vextreme-rescue #PWR0148
 U 1 1 5E24168D
 P 9450 5650
@@
 $EndComp
 $Comp
-L vextreme-rescue:GND-vextreme-rescue #PWR0147
+L vextreme-rescue:GND-vextreme-rescue-vextreme-rescue #PWR0147
 U 1 1 5E241687
 P 9450 6250
@@
 $EndComp
 $Comp
-L vextreme-rescue:GND-vextreme-rescue #PWR0143
+L vextreme-rescue:GND-vextreme-rescue-vextreme-rescue #PWR0143
 U 1 1 5E237D78
 P 8750 6250
@@
 $EndComp
 $Comp
-L vextreme-rescue:+5V-vextreme-rescue #PWR0144
+L vextreme-rescue:+5V-vextreme-rescue-vextreme-rescue #PWR0144
 U 1 1 5E237D7E
 P 8750 5650
@@
 	10450 5850 10650 5850
 $Comp
-L vextreme-rescue:GND-vextreme-rescue #PWR0133
+L vextreme-rescue:GND-vextreme-rescue-vextreme-rescue #PWR0133
 U 1 1 5EEAFF3A
 P 10500 5550
@@
 	1900 6850 1900 6800
 $Comp
-L vextreme-rescue:GND-vextreme-rescue #PWR01
+L vextreme-rescue:GND-vextreme-rescue-vextreme-rescue #PWR01
 U 1 1 5EE9BB2A
 P 2100 7350
@@
 	10350 5000 10650 5000
 $Comp
-L vextreme-rescue:+5V-vextreme-rescue #PWR0135
+L vextreme-rescue:+5V-vextreme-rescue-vextreme-rescue #PWR0135
 U 1 1 60A19939
 P 10350 4900
@@
 $EndComp
 Text Notes 7950 3500 0    50   ~ 0
-v0.5 Changelog\n——————————————————————\n- Added a location for the Wi-Fi Module\n- Changed J2 to support +5V for the Wi-Fi Module\n- Changed the artwork a bit and side up/down text.
+v0.5 Changelog (aka v1.0)\n——————————————————————\n- Added a location for the Wi-Fi Module\n- Changed J2 to support +5V for the Wi-Fi Module\n- Changed the artwork a bit and side up/down text.
 $EndSCHEMATC
